Commit message: fix (?) spot_description to have arm

File: spot_description/urdf/spot.urdf.xacro (robot description, xacro)
@@ -261,4 +261,6 @@
     <!-- Standard accessories. -->
     <xacro:include filename="$(find spot_description)/urdf/accessories.urdf.xacro" />
+    <!-- arm. -->
+    <xacro:include filename="$(find spot_description)/urdf/spot_arm.urdf.xacro" />
     <!-- Optional custom includes. -->
     <xacro:include filename="$(optenv SPOT_URDF_EXTRAS empty.urdf)" />

File: spot_description/urdf/spot_arm.urdf.xacro (robot description, xacro)
@@ -1,196 +1,9 @@
-<robot name="spot">
-  <link name="base">
-    <visual>
-      <origin xyz="0 0 0" rpy="0 0 0"/>
-      <geometry>
-        <mesh filename="link_models/base.obj"/>
-      </geometry>
-<material name="base"> <color rgba="1 0.8431 0 1"/></material>    </visual>
-  </link>
-  <link name="fl.hip">
-    <visual>
-      <origin xyz="0 0 0" rpy="0 0 0"/>
-      <geometry>
-        <mesh filename="link_models/fl.hip.obj"/>
-      </geometry>
-<material name="fl.hip"> <color rgba="0.2 0.2 0.2 1"/></material>    </visual>
-  </link>
-  <joint name="fl.hx" type="revolute">
-    <origin xyz="0.29785 0.05500 0.00000" rpy="0 0 0"/>
-    <axis xyz="1 0 0"/>
-    <parent link="base"/>
-    <child link="fl.hip"/>
-     <limit effort="1000" velocity="1000.00" lower="-0.791936" upper="0.783921"/>
-  </joint>
-  <link name="fl.uleg">
-    <visual>
-      <origin xyz="0 0 0" rpy="0 0 0"/>
-      <geometry>
-        <mesh filename="link_models/fl.uleg.obj"/>
-      </geometry>
-<material name="fl.uleg"> <color rgba="1 0.8431 0 1"/></material>    </visual>
-  </link>
-  <joint name="fl.hy" type="revolute">
-    <origin xyz="0.0 0.110945 0.0" rpy="0 0 0"/>
-    <axis xyz="0 1      0"/>
-    <parent link="fl.hip"/>
-    <child link="fl.uleg"/>
-     <limit effort="1000" velocity="1000.00" lower="-0.872867" upper="2.26796"/>
-  </joint>
-  <link name="fl.lleg">
-    <visual>
-      <origin xyz="0 0 0" rpy="0 0 0"/>
-      <geometry>
-        <mesh filename="link_models/fl.lleg.obj"/>
-      </geometry>
-<material name="fl.lleg"> <color rgba="0.2 0.2 0.2 1"/></material>    </visual>
-  </link>
-  <joint name="fl.kn" type="revolute">
-    <origin xyz="0.025 0.000 -0.3205" rpy="0 0 0"/>
-    <axis xyz="0 1 0"/>
-    <parent link="fl.uleg"/>
-    <child link="fl.lleg"/>
-     <limit effort="1000" velocity="1000.00" lower="-2.79243" upper="-0.293192"/>
-  </joint>
-  <link name="fr.hip">
-    <visual>
-      <origin xyz="0 0 0" rpy="0 0 0"/>
-      <geometry>
-        <mesh filename="link_models/fr.hip.obj"/>
-      </geometry>
-<material name="fr.hip"> <color rgba="0.2 0.2 0.2 1"/></material>    </visual>
-  </link>
-  <joint name="fr.hx" type="revolute">
-    <origin xyz="0.29785 -0.05500 0.00000" rpy="0 0 0"/>
-    <axis xyz="1 0 0"/>
-    <parent link="base"/>
-    <child link="fr.hip"/>
-     <limit effort="1000" velocity="1000.00" lower="-0.772064" upper="0.800867"/>
-  </joint>
-  <link name="fr.uleg">
-    <visual>
-      <origin xyz="0 0 0" rpy="0 0 0"/>
-      <geometry>
-        <mesh filename="link_models/fr.uleg.obj"/>
-      </geometry>
-<material name="fr.uleg"> <color rgba="1 0.8431 0 1"/></material>    </visual>
-  </link>
-  <joint name="fr.hy" type="revolute">
-    <origin xyz="0.0 -0.110945 0.0" rpy="0 0 0"/>
-    <axis xyz="0  1      0"/>
-    <parent link="fr.hip"/>
-    <child link="fr.uleg"/>
-     <limit effort="1000" velocity="1000.00" lower="-0.878417" upper="2.26234"/>
-  </joint>
-  <link name="fr.lleg">
-    <visual>
-      <origin xyz="0 0 0" rpy="0 0 0"/>
-      <geometry>
-        <mesh filename="link_models/fr.lleg.obj"/>
-      </geometry>
-<material name="fr.lleg"> <color rgba="0.2 0.2 0.2 1"/></material>    </visual>
-  </link>
-  <joint name="fr.kn" type="revolute">
-    <origin xyz="0.025 0.000 -0.3205" rpy="0 0 0"/>
-    <axis xyz="0 1 0"/>
-    <parent link="fr.uleg"/>
-    <child link="fr.lleg"/>
-     <limit effort="1000" velocity="1000.00" lower="-2.78721" upper="-0.283179"/>
-  </joint>
-  <link name="hl.hip">
-    <visual>
-      <origin xyz="0 0 0" rpy="0 0 0"/>
-      <geometry>
-        <mesh filename="link_models/hl.hip.obj"/>
-      </geometry>
-<material name="hl.hip"> <color rgba="0.2 0.2 0.2 1"/></material>    </visual>
-  </link>
-  <joint name="hl.hx" type="revolute">
-    <origin xyz="-0.29785 0.05500 0.00000" rpy="0 0 0"/>
-    <axis xyz="1 0 0"/>
-    <parent link="base"/>
-    <child link="hl.hip"/>
-     <limit effort="1000" velocity="1000.00" lower="-0.791525" upper="0.778251"/>
-  </joint>
-  <link name="hl.uleg">
-    <visual>
-      <origin xyz="0 0 0" rpy="0 0 0"/>
-      <geometry>
-        <mesh filename="link_models/hl.uleg.obj"/>
-      </geometry>
-<material name="hl.uleg"> <color rgba="1 0.8431 0 1"/></material>    </visual>
-  </link>
-  <joint name="hl.hy" type="revolute">
-    <origin xyz="0.0 0.110945 0.0" rpy="0 0 0"/>
-    <axis xyz="0 1      0"/>
-    <parent link="hl.hip"/>
-    <child link="hl.uleg"/>
-     <limit effort="1000" velocity="1000.00" lower="-0.877249" upper="2.26246"/>
-  </joint>
-  <link name="hl.lleg">
-    <visual>
-      <origin xyz="0 0 0" rpy="0 0 0"/>
-      <geometry>
-        <mesh filename="link_models/hl.lleg.obj"/>
-      </geometry>
-<material name="hl.lleg"> <color rgba="0.2 0.2 0.2 1"/></material>    </visual>
-  </link>
-  <joint name="hl.kn" type="revolute">
-    <origin xyz="0.025 0.000 -0.3205" rpy="0 0 0"/>
-    <axis xyz="0 1 0"/>
-    <parent link="hl.uleg"/>
-    <child link="hl.lleg"/>
-     <limit effort="1000" velocity="1000.00" lower="-2.79237" upper="-0.277268"/>
-  </joint>
-  <link name="hr.hip">
-    <visual>
-      <origin xyz="0 0 0" rpy="0 0 0"/>
-      <geometry>
-        <mesh filename="link_models/hr.hip.obj"/>
-      </geometry>
-<material name="hr.hip"> <color rgba="0.2 0.2 0.2 1"/></material>    </visual>
-  </link>
-  <joint name="hr.hx" type="revolute">
-    <origin xyz="-0.29785 -0.05500 0.00000" rpy="0 0 0"/>
-    <axis xyz="1 0 0"/>
-    <parent link="base"/>
-    <child link="hr.hip"/>
-     <limit effort="1000" velocity="1000.00" lower="-0.787378" upper="0.785509"/>
-  </joint>
-  <link name="hr.uleg">
-    <visual>
-      <origin xyz="0 0 0" rpy="0 0 0"/>
-      <geometry>
-        <mesh filename="link_models/hr.uleg.obj"/>
-      </geometry>
-<material name="hr.uleg"> <color rgba="1 0.8431 0 1"/></material>    </visual>
-  </link>
-  <joint name="hr.hy" type="revolute">
-    <origin xyz="0.0 -0.110945 0.0" rpy="0 0 0"/>
-    <axis xyz="0  1      0"/>
-    <parent link="hr.hip"/>
-    <child link="hr.uleg"/>
-     <limit effort="1000" velocity="1000.00" lower="-0.898918" upper="2.2403"/>
-  </joint>
-  <link name="hr.lleg">
-    <visual>
-      <origin xyz="0 0 0" rpy="0 0 0"/>
-      <geometry>
-        <mesh filename="link_models/hr.lleg.obj"/>
-      </geometry>
-<material name="hr.lleg"> <color rgba="0.2 0.2 0.2 1"/></material>    </visual>
-  </link>
-  <joint name="hr.kn" type="revolute">
-    <origin xyz="0.025 0.000 -0.3205" rpy="0 0 0"/>
-    <axis xyz="0 1 0"/>
-    <parent link="hr.uleg"/>
-    <child link="hr.lleg"/>
-     <limit effort="1000" velocity="1000.00" lower="-2.79286" upper="-0.286494"/>
-  </joint>
+<?xml version="1.0" ?>
+<robot name="spot" xmlns:xacro="http://www.ros.org/wiki/xacro">
   <link name="arm0.link_sh0">
     <visual>
       <origin xyz="0 0 0" rpy="0 0 0"/>
       <geometry>
-        <mesh filename="link_models/arm0.link_sh0.obj"/>
+        <mesh filename="package://spot_description/meshes/arm/arm0.link_sh0.obj"/>
       </geometry>
 <material name="arm0.link_sh0"> <color rgba="0.2 0.2 0.2 1"/></material>    </visual>
@@ -199,5 +12,5 @@
     <origin xyz="0.292 0.0 0.188" rpy="0 0 0"/>
     <axis xyz="0 0 1"/>
-    <parent link="base"/>
+    <parent link="body"/>
     <child link="arm0.link_sh0"/>
      <limit effort="1000" velocity="1000.00" lower="-2.61799387799149441136" upper="3.14159265358979311599"/>
@@ -207,5 +20,5 @@
       <origin xyz="0 0 0" rpy="0 0 0"/>
       <geometry>
-        <mesh filename="link_models/arm0.link_sh1.obj"/>
+        <mesh filename="package://spot_description/meshes/arm/arm0.link_sh1.obj"/>
       </geometry>
 <material name="arm0.link_sh1"> <color rgba="0.2 0.2 0.2 1"/></material>    </visual>
@@ -222,5 +35,5 @@
       <origin xyz="0 0 0" rpy="0 0 0"/>
       <geometry>
-        <mesh filename="link_models/arm0.link_hr0.obj"/>
+        <mesh filename="package://spot_description/meshes/arm/arm0.link_hr0.obj"/>
       </geometry>
 <material name="arm0.link_hr0"> <color rgba="0.2 0.2 0.2 1"/></material>    </visual>
@@ -237,5 +50,5 @@
       <origin xyz="0 0 0" rpy="0 0 0"/>
       <geometry>
-        <mesh filename="link_models/arm0.link_el0.obj"/>
+        <mesh filename="package://spot_description/meshes/arm/arm0.link_el0.obj"/>
       </geometry>
 <material name="arm0.link_el0"> <color rgba="0.2 0.2 0.2 1"/></material>    </visual>
@@ -252,5 +65,5 @@
       <origin xyz="0 0 0" rpy="0 0 0"/>
       <geometry>
-        <mesh filename="link_models/arm0.link_el1.obj"/>
+        <mesh filename="package://spot_description/meshes/arm/arm0.link_el1.obj"/>
       </geometry>
 <material name="arm0.link_el1"> <color rgba="0.2 0.2 0.2 1"/></material>    </visual>
@@ -267,5 +80,5 @@
       <origin xyz="0 0 0" rpy="0 0 0"/>
       <geometry>
-        <mesh filename="link_models/arm0.link_wr0.obj"/>
+        <mesh filename="package://spot_description/meshes/arm/arm0.link_wr0.obj"/>
       </geometry>
 <material name="arm0.link_wr0"> <color rgba="0.2 0.2 0.2 1"/></material>    </visual>
@@ -282,5 +95,5 @@
       <origin xyz="0 0 0" rpy="0 0 0"/>
       <geometry>
-        <mesh filename="link_models/arm0.link_wr1.obj"/>
+        <mesh filename="package://spot_description/meshes/arm/arm0.link_wr1.obj"/>
       </geometry>
 <material name="arm0.link_wr1"> <color rgba="0.2 0.2 0.2 1"/></material>    </visual>
@@ -297,5 +110,5 @@
       <origin xyz="0 0 0" rpy="0 0 0"/>
       <geometry>
-        <mesh filename="link_models/arm0.link_fngr.obj"/>
+        <mesh filename="package://spot_description/meshes/arm/arm0.link_fngr.obj"/>
       </geometry>
 <material name="arm0.link_fngr"> <color rgba="0.2 0.2 0.2 1"/></material>    </visual>
